File: _restore_backup_2026-05-13T08-43-48-773/hexboard.kicad_sch (KiCad schematic)
At the start: 49 parts, among them J1 USB_C_Receptacle_USB2.0_16P, J2 USB_A, J3 Conn_01x20, J4 Conn_01x20, J5 Conn_01x04, SW1 SW_Push, SW2 SW_Push, SW3 SW_Push, U1 RP2040, U2 MCP1700x-330xxTT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

Commit message: added design on back and added a few more things
Parts:
- removed C7: 0.1uF, u3, symbol Device:C
- removed D2: LED, LED_SMD:LED_0402_1005Metric, symbol Device:LED
- removed D3: WS2812B, LED_SMD:LED_WS2812B_PLCC4_5.0x5.0mm_P3.2mm, symbol LED:WS2812B
- removed J5: Conn_01x04, Connector_PinHeader_2.54mm:PinHeader_1x04_P2.54mm_Vertical, symbol Connector_Generic:Conn_01x04
- removed R10, R11: 4.7K, Resistor_SMD:R_0402_1005Metric, symbol Device:R
- removed R12: 10K, Resistor_SMD:R_0402_1005Metric, symbol Device:R
- removed R13: 100 ohm, Resistor_SMD:R_0402_1005Metric, symbol Device:R
- removed SW3: SW_Push, Button_Switch_SMD:SW_SPST_B3S-1000, symbol Switch:SW_Push
- removed TP1: TESTVBUS, TestPoint:TestPoint_Pad_1.0x1.0mm, symbol Connector:TestPoint
- removed TP2: TEST_3V3, TestPoint:TestPoint_Pad_1.0x1.0mm, symbol Connector:TestPoint
- removed TP3: TESTGND, TestPoint:TestPoint_Pad_1.0x1.0mm, symbol Connector:TestPoint
- removed TP4: TESTSCL, TestPoint:TestPoint_Pad_1.0x1.0mm, symbol Connector:TestPoint
- removed TP5: TESTSDA, TestPoint:TestPoint_Pad_1.0x1.0mm, symbol Connector:TestPoint
- removed U4: TMP102xxDRL, Package_TO_SOT_SMD:SOT-563, symbol Sensor_Temperature:TMP102xxDRL
- U3: footprint Package_SO:SOIC-8_3.9x4.9mm_P1.27mm -> Package_SON:Winbond_USON-8-1EP_3x2mm_P0.5mm_EP0.2x1.6mm
Connections:
- net I2C_SCL: no longer names the net of J3.6 (Pin_6), U1.7 (GPIO5)
- net I2C_SDA: no longer names the net of J3.5 (Pin_5), U1.6 (GPIO4)
- net RGB_DIN: no longer names the net of J3.9 (Pin_9), U1.11 (GPIO8)
- net USR_BTN: no longer names the net of J3.7 (Pin_7), U1.8 (GPIO6)
- net USR_LED: no longer names the net of J3.8 (Pin_8), U1.9 (GPIO7)
- no-connect marks 5 -> 4
Other:
- moved on the sheet: J3, J4
