File: _restore_backup_2026-05-13T09-51-41-049/hexboard.kicad_sch (KiCad schematic)
At the start: 49 parts, among them J1 USB_C_Receptacle_USB2.0_16P, J2 USB_A, J3 Conn_01x20, J4 Conn_01x20, J5 Conn_01x04, SW1 SW_Push, SW2 SW_Push, SW3 SW_Push, U1 RP2040, U2 MCP1700x-330xxTT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

Commit message: added design on back and added a few more things
Parts:
- removed C7: 0.1uF, u3, symbol Device:C
- removed D3: WS2812B, LED_SMD:LED_WS2812B_PLCC4_5.0x5.0mm_P3.2mm, symbol LED:WS2812B
- removed U4: TMP102xxDRL, Package_TO_SOT_SMD:SOT-563, symbol Sensor_Temperature:TMP102xxDRL
- U3: footprint Package_SO:SOIC-8_3.9x4.9mm_P1.27mm -> Package_SON:Winbond_USON-8-1EP_3x2mm_P0.5mm_EP0.2x1.6mm
Connections:
- net RGB_DIN: no longer names the net of J3.9 (Pin_9), U1.11 (GPIO8)
- no-connect marks 5 -> 4
